File: Proyecto-Ecosistema-Sensor-de-Temperatura/KiCad/proyecto sensor temperatura.kicad_sch (KiCad schematic)
At the start: 6 parts

Commit message: Importar contenido de proyecto-sensor-temperatura-humedad a main
Connections:
- net GND: now also Micro_controlador.14 (GND)
Other:
- moved on the sheet: H1, H2, H3, H4
Changed lines of the file:
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@@
+    (stroke (width 0) (type default) (color 0 0 0 0))
+  )
+  (wire (pts (xy 60.96 112.395) (xy 56.515 112.395))
     (stroke (width 0) (type default) (color 0 0 0 0))
   )
@@
   )
   (wire (pts (xy 88.9 109.855) (xy 92.075 109.855))
+    (stroke (width 0) (type default) (color 0 0 0 0))
+  )
+  (wire (pts (xy 56.515 112.395) (xy 56.515 113.665))
     (stroke (width 0) (type default) (color 0 0 0 0))
   )
@@
     (effects (font (size 1.27 1.27)) (justify left bottom))
   )
-  (symbol (lib_id "Mechanical:MountingHole") (at 25.654 157.226 0) (unit 1)
+  (symbol (lib_id "Mechanical:MountingHole") (at -20.32 147.066 0) (unit 1)
     (in_bom yes) (on_board yes) (fields_autoplaced)
-    (property "Reference" "H3" (id 0) (at 28.194 155.9559 0)
+    (property "Reference" "H3" (id 0) (at -17.78 145.7959 0)
       (effects (font (size 1.27 1.27)) (justify left))
     )
-    (property "Value" "MountingHole" (id 1) (at 28.194 158.4959 0)
+    (property "Value" "MountingHole" (id 1) (at -17.78 148.3359 0)
       (effects (font (size 1.27 1.27)) (justify left))
     )
-    (property "Footprint" "EESTN5:Separador_M3_5mm" (id 2) (at 25.654 157.226 0)
-      (effects (font (size 1.27 1.27)) hide)
-    )
-    (property "Datasheet" "~" (id 3) (at 25.654 157.226 0)
+    (property "Footprint" "EESTN5:Separador_M3_5mm" (id 2) (at -20.32 147.066 0)
+      (effects (font (size 1.27 1.27)) hide)
+    )
+    (property "Datasheet" "~" (id 3) (at -20.32 147.066 0)
       (effects (font (size 1.27 1.27)) hide)
     )
@@
     (pin "1")
   )
-  (symbol (lib_id "Mechanical:MountingHole") (at 25.654 147.066 0) (unit 1)
+  (symbol (lib_id "Mechanical:MountingHole") (at -20.32 136.906 0) (unit 1)
     (in_bom yes) (on_board yes) (fields_autoplaced)
-    (property "Reference" "H1" (id 0) (at 28.194 145.7959 0)
+    (property "Reference" "H1" (id 0) (at -17.78 135.6359 0)
       (effects (font (size 1.27 1.27)) (justify left))
     )
-    (property "Value" "MountingHole" (id 1) (at 28.194 148.3359 0)
+    (property "Value" "MountingHole" (id 1) (at -17.78 138.1759 0)
       (effects (font (size 1.27 1.27)) (justify left))
     )
-    (property "Footprint" "EESTN5:Separador_M3_5mm" (id 2) (at 25.654 147.066 0)
-      (effects (font (size 1.27 1.27)) hide)
-    )
-    (property "Datasheet" "~" (id 3) (at 25.654 147.066 0)
+    (property "Footprint" "EESTN5:Separador_M3_5mm" (id 2) (at -20.32 136.906 0)
+      (effects (font (size 1.27 1.27)) hide)
+    )
+    (property "Datasheet" "~" (id 3) (at -20.32 136.906 0)
       (effects (font (size 1.27 1.27)) hide)
     )
@@
     (pin "1")
   )
-  (symbol (lib_id "Mechanical:MountingHole") (at 25.654 162.306 0) (unit 1)
+  (symbol (lib_id "Mechanical:MountingHole") (at -20.32 152.146 0) (unit 1)
     (in_bom yes) (on_board yes) (fields_autoplaced)
-    (property "Reference" "H4" (id 0) (at 28.194 161.0359 0)
+    (property "Reference" "H4" (id 0) (at -17.78 150.8759 0)
       (effects (font (size 1.27 1.27)) (justify left))
     )
-    (property "Value" "MountingHole" (id 1) (at 28.194 163.5759 0)
+    (property "Value" "MountingHole" (id 1) (at -17.78 153.4159 0)
       (effects (font (size 1.27 1.27)) (justify left))
     )
-    (property "Footprint" "EESTN5:Separador_M3_5mm" (id 2) (at 25.654 162.306 0)
-      (effects (font (size 1.27 1.27)) hide)
-    )
-    (property "Datasheet" "~" (id 3) (at 25.654 162.306 0)
-      (effects (font (size 1.27 1.27)) hide)
-    )
-  )
-  (symbol (lib_id "Mechanical:MountingHole") (at 25.654 152.146 0) (unit 1)
+    (property "Footprint" "EESTN5:Separador_M3_5mm" (id 2) (at -20.32 152.146 0)
+      (effects (font (size 1.27 1.27)) hide)
+    )
+    (property "Datasheet" "~" (id 3) (at -20.32 152.146 0)
+      (effects (font (size 1.27 1.27)) hide)
+    )
+  )
+  (symbol (lib_id "Mechanical:MountingHole") (at -20.32 141.986 0) (unit 1)
     (in_bom yes) (on_board yes) (fields_autoplaced)
-    (property "Reference" "H2" (id 0) (at 28.194 150.8759 0)
+    (property "Reference" "H2" (id 0) (at -17.78 140.7159 0)
       (effects (font (size 1.27 1.27)) (justify left))
     )
-    (property "Value" "MountingHole" (id 1) (at 28.194 153.4159 0)
+    (property "Value" "MountingHole" (id 1) (at -17.78 143.2559 0)
       (effects (font (size 1.27 1.27)) (justify left))
     )
-    (property "Footprint" "EESTN5:Separador_M3_5mm" (id 2) (at 25.654 152.146 0)
-      (effects (font (size 1.27 1.27)) hide)
-    )
-    (property "Datasheet" "~" (id 3) (at 25.654 152.146 0)
-      (effects (font (size 1.27 1.27)) hide)
-    )
+    (property "Footprint" "EESTN5:Separador_M3_5mm" (id 2) (at -20.32 141.986 0)
+      (effects (font (size 1.27 1.27)) hide)
+    )
+    (property "Datasheet" "~" (id 3) (at -20.32 141.986 0)
+      (effects (font (size 1.27 1.27)) hide)
+    )
